Commit message: URDF arm fixed to ground added

File: manipulation/scorbot_description/urdf/arm_fixed_to_ground.xacro (robot description, xacro)
@@ -48,5 +48,5 @@
   <xacro:macro name="scorbot" params="prefix parent *origin">
     <!-- WORLD LINK -> Used for fixing robot to Gazebo '${prefix}_base_link' -->
-    <!-- <link name="world"/> -->
+    <link name="world"/>
     <joint name="${prefix}_base_joint" type="fixed">
       <xacro:insert_block name="origin"/>

File: rover_autonav/urdf/cali_fixed_to_ground.xacro (robot description, xacro)
@@ -3,5 +3,5 @@
        name="ur3e" >
   <!-- ARM -->
-  <xacro:include filename="$(find manipulation)/scorbot_description/urdf/scorbot_v3.xacro" />
+  <xacro:include filename="$(find manipulation)/scorbot_description/urdf/arm_fixed_to_ground.xacro" />
   <!-- Here we create the Xacro macro to attach the Gripper to the arm_link-->
   <xacro:scorbot prefix="scorbot" parent="world">
