Commit message: URDF fixed

File: manipulation/scorbot_description/urdf/scorbot_v3.xacro (robot description, xacro)
@@ -7,6 +7,6 @@
   <xacro:macro name="scorbot" params="prefix parent *origin">
     <!-- Used for fixing robot to Gazebo 'base_link' -->
-    <!-- <link name="world"/>
-    <joint name="fixed" type="fixed">
+    <link name="world"/>
+    <!-- <joint name="fixed" type="fixed">
       <parent link="world"/>
       <child link="base_link"/>
@@ -81,5 +81,5 @@
       <origin xyz="0 0 0.2274" rpy="0 0 0"/>
       <axis xyz="0 0 1"/>
-      <limit lower="-5.4105207" upper="5.4105207" effort="0" velocity="2"/>
+      <limit lower="-3.1415926535897931" upper="3.1415926535897931" effort="1000" velocity="2"/>
     </joint>
     <!--Link 2 ELBOW LINK-->
@@ -118,5 +118,5 @@
       <origin xyz="0.0255 0 0.13" rpy="-1.570796327 -1.570796327 0"/>
       <axis xyz="0 0 1"/>
-      <limit lower="-0.610865" upper="2.268928" effort="0" velocity="2"/>
+      <limit lower="-0.610865" upper="2.268928" effort="1000" velocity="2"/>
       <!-- <dynamics
         damping="0.0"

File: rover_autonav/urdf/cali_fixed_to_ground.xacro (robot description, xacro)
@@ -2,18 +2,8 @@
 <robot xmlns:xacro="http://ros.org/wiki/xacro"
        name="ur3e" >
-  <!-- common stuff -->
-  <!-- <xacro:include filename="$(find ur_e_description)/urdf/rosbob.gazebo" /> -->
-  <!-- MOBILE ROBOT -->
-  <!-- NO MESH FOR MOBILE ROBOT-->
-  <!-- <xacro:include filename="$(find rover_autonav)/urdf/rosbob_v2.xacro" /> -->
-  <!-- MESH FOR MOBILE ROBOT-->
-  <xacro:include filename="$(find rover_autonav)/urdf/world.xacro" />
   <!-- ARM -->
   <xacro:include filename="$(find manipulation)/scorbot_description/urdf/scorbot_v3.xacro" />
   <!-- Here we create the Xacro macro to attach the Gripper to the arm_link-->
-  <xacro:scorbot prefix="scorbot" parent="arm_link">
-    <!-- NO MESH FOR MOBILE ROBOT-->
-    <!-- <origin xyz="0.0 0 0.43" rpy="0 0 0" /> -->
-    <!-- MESH FOR MOBILE ROBOT-->
+  <xacro:scorbot prefix="scorbot" parent="world">
     <origin xyz="0.0 0 0.0" rpy="0 0 0" />
   </xacro:scorbot>

Commit message: URDF arm updated: xacro for inertias

File: manipulation/scorbot_description/urdf/scorbot_v3.xacro (robot description, xacro)
@@ -5,4 +5,47 @@
   <xacro:property name="d435_cam_depth" value="0.025"/>
   <xacro:property name="d435_cam_height" value="0.025"/>
+  <!--Masses values for each link-->
+  <xacro:property name="mass_base_link" value="7.0" />
+  <xacro:property name="mass_link_1" value="6.0" />
+  <xacro:property name="mass_link_2" value="1.0" />
+  <xacro:property name="mass_link_3" value="1.0" />
+  <xacro:property name="mass_link_4" value="0.1" />
+  <xacro:property name="mass_link_5" value="0.1" />
+  <xacro:property name="mass_pad1_Link" value="1.0" />
+  <xacro:property name="mass_pad2_Link" value="1.0" />
+  <!--Surrounding boxes values for each link-->
+  <xacro:property name="base_link_x" value="0.24" />
+  <xacro:property name="base_link_y" value="0.24" />
+  <xacro:property name="base_link_z" value="0.2274" />
+  <xacro:property name="link_1_x" value="0.205" />
+  <xacro:property name="link_1_y" value="0.26" />
+  <xacro:property name="link_1_z" value="0.17" />
+  <xacro:property name="link_2_x" value="0.28749" />
+  <xacro:property name="link_2_y" value="0.069982" />
+  <xacro:property name="link_2_z" value="0.169" />
+  <xacro:property name="link_3_x" value="0.289918" />
+  <xacro:property name="link_3_y" value="0.06" />
+  <xacro:property name="link_3_z" value="0.15" />
+  <xacro:property name="link_4_x" value="0.183046" />
+  <xacro:property name="link_4_y" value="0.073212" />
+  <xacro:property name="link_4_z" value="0.075543" />
+  <xacro:property name="link_5_x" value="0.06" />
+  <xacro:property name="link_5_y" value="0.14" />
+  <xacro:property name="link_5_z" value="0.238" />
+<!--
+  <xacro:property name="pad1_link_x" value="1.0" />
+  <xacro:property name="pad1_link_y" value="1.0" />
+  <xacro:property name="pad1_link_z" value="0.1" />
+  <xacro:property name="pad2_link_x" value="1.0" />
+  <xacro:property name="pad2_link_y" value="1.0" />
+  <xacro:property name="pad2_link_z" value="0.1" />
+   -->
+  <!--Inertia Calculator for a Box-->
+  <xacro:macro name="box_inertia" params="mass x y z">
+    <inertia  ixx="${mass*(y*y+z*z)/12.0}" ixy = "0" ixz = "0"
+              iyy="${mass*(x*x+z*z)/12.0}" iyz = "0"
+              izz="${mass*(x*x+y*y)/12.0}"
+    />
+  </xacro:macro>
   <xacro:macro name="scorbot" params="prefix parent *origin">
     <!-- Used for fixing robot to Gazebo 'base_link' -->
@@ -25,6 +68,7 @@
           rpy="0 0 0" />
         <mass
-          value="7" />
-        <inertia
+          value="${mass_base_link}" />
+        <xacro:box_inertia mass="${mass_base_link}" x="${base_link_x}" y="${base_link_y}" z="${base_link_z}"/>
+        <!-- <inertia
           ixx="0.06376461"
           ixy="0.0"
@@ -32,5 +76,5 @@
           iyy="0.06376461"
           iyz="0.0"
-          izz="0.0672" />
+          izz="0.0672" /> -->
       </inertial>
       <visual>
@@ -39,10 +83,10 @@
         </geometry>
       </visual>
-      <!-- <collision>
+      <collision>
         <origin xyz="0 0 0" rpy="0 0 0"/>
         <geometry>
           <mesh filename="package://manipulation/scorbot_description/meshes/visual/Parte_1(1).DAE"/>
         </geometry>
-      </collision> -->
+      </collision>
     </link>
     <!--Link 1 SHOULDER LINK-->
@@ -54,6 +98,7 @@
           rpy="0 0 0" />
         <mass
-          value="6" />
-        <inertia
+          value="${mass_link_1}" />
+        <xacro:box_inertia mass="${mass_link_1}" x="${link_1_x}" y="${link_1_y}" z="${link_1_z}"/>
+        <!-- <inertia
           ixx="0.04825000000000001"
           ixy="0.0"
@@ -61,5 +106,5 @@
           iyy="0.0354625"
           iyz="0.0"
-          izz="0.0548125" />
+          izz="0.0548125" /> -->
       </inertial>
       <visual>
@@ -68,10 +113,10 @@
         </geometry>
       </visual>
-      <!-- <collision>
+      <collision>
         <origin xyz="0 0 0" rpy="0 0 0"/>
         <geometry>
           <mesh filename="package://manipulation/scorbot_description/meshes/visual/Parte_2(1)x.DAE"/>
         </geometry>
-      </collision> -->
+      </collision>
     </link>
     <!--Joint 1 BASE JOINT-->
@@ -91,6 +136,7 @@
           rpy="0 0 0" />
         <mass
-          value="1" />
-        <inertia
+          value="${mass_link_2}" />
+        <xacro:box_inertia mass="${mass_link_2}" x="${link_2_x}" y="${link_2_y}" z="${link_2_z}"/>
+        <!-- <inertia
           ixx="0.002788206693666667"
           ixy="0.0"
@@ -98,5 +144,5 @@
           iyy="0.009267625008333334"
           iyz="0.0"
-          izz="0.007295665035333334" />
+          izz="0.007295665035333334" /> -->
     </inertial>
       <visual>
@@ -105,10 +151,10 @@
         </geometry>
       </visual>
-      <!-- <collision>
+      <collision>
         <origin xyz="0 0 0" rpy="0 0 0"/>
         <geometry>
           <mesh filename="package://manipulation/scorbot_description/meshes/visual/Parte_3(2)x.DAE"/>
         </geometry>
-      </collision> -->
+      </collision>
     </link>
     <!--Joint 2 SHOULDER JOINT-->
@@ -125,5 +171,5 @@
     <!--Link 3 PITCH LINK-->
     <!-- Bounding box: 0.289918 0.06 0.15 -->
-    <!-- <link name="${prefix}_link_3">
+    <link name="${prefix}_link_3">
       <inertial>
         <origin
@@ -131,6 +177,7 @@
           rpy="0 0 0" />
         <mass
-          value="1" />
-        <inertia
+          value="${mass_link_3}" />
+        <xacro:box_inertia mass="${mass_link_3}" x="${link_3_x}" y="${link_3_y}" z="${link_3_z}"/>
+        <!-- <inertia
           ixx="0.002175"
           ixy="0.0"
@@ -138,5 +185,5 @@
           iyy="0.008879370560333333"
           iyz="0.0"
-          izz="0.007304370560333334" />
+          izz="0.007304370560333334" /> -->
     </inertial>
       <visual>
@@ -151,19 +198,19 @@
         </geometry>
       </collision>
-    </link> -->
+    </link>
     <!--Joint 3 ELBOW JOINT-->
-    <!-- <joint name="${prefix}_joint_3" type="revolute">
+    <joint name="${prefix}_joint_3" type="revolute">
       <parent link="${prefix}_link_2"/>
       <child link="${prefix}_link_3"/>
       <origin xyz="0.2225 0 0" rpy="0 0 0"/>
       <axis xyz="0 0 1"/>
-      <limit lower="-2.268928" upper="2.268928" effort="0" velocity="2"/>
-      <dynamics
+      <limit lower="-2.268928" upper="2.268928" effort="1000" velocity="2"/>
+      <!-- <dynamics
         damping="0.0"
-        friction="0.5" />
-    </joint> -->
+        friction="0.5" /> -->
+    </joint>
     <!--Link 4 ROLL LINK-->
     <!-- Bounding box: 0.183046 0.073212 0.075543 -->
-    <!-- <link name="${prefix}_link_4">
+    <link name="${prefix}_link_4">
       <inertial>
         <origin
@@ -171,6 +218,7 @@
           rpy="0 0 0" />
         <mass
-          value="0.1" />
-        <inertia
+          value="${mass_link_4}" />
+        <xacro:box_inertia mass="${mass_link_4}" x="${link_4_x}" y="${link_4_y}" z="${link_4_z}"/>
+        <!-- <inertia
           ixx="9.2222848275e-05"
           ixy="0.0"
@@ -178,5 +226,5 @@
           iyy="0.0003267715247083333"
           iyz="0.0"
-          izz="0.0003238819588333333" />
+          izz="0.0003238819588333333" /> -->
     </inertial>
       <visual>
@@ -192,19 +240,19 @@
         </geometry>
       </collision>
-    </link> -->
+    </link>
     <!--Joint 4 PITCH JOINT-->
-    <!-- <joint name="${prefix}_joint_4" type="revolute">
+    <joint name="${prefix}_joint_4" type="revolute">
       <parent link="${prefix}_link_3"/>
       <child link="${prefix}_link_4"/>
       <origin xyz="0.2225 0 0" rpy="0 0 0"/>
       <axis xyz="0 0 1"/>
-      <limit lower="-2.268928" upper="2.268928" effort="0" velocity="2"/>
-      <dynamics
+      <limit lower="-2.268928" upper="2.268928" effort="1000" velocity="2"/>
+      <!-- <dynamics
         damping="0.0"
-        friction="0.5" />
-    </joint> -->
+        friction="0.5" /> -->
+    </joint>
     <!--Link 5 GRIPPER LINK-->
     <!-- Bounding box: 0.06 0.14 0.238 -->
-    <!-- <link name="${prefix}_link_5">
+    <link name="${prefix}_link_5">
       <inertial>
         <origin
@@ -212,6 +260,7 @@
           rpy="0 0 0" />
         <mass
-          value="0.1" />" />
-        <inertia
+          value="${mass_link_5}" />" />
+        <xacro:box_inertia mass="${mass_link_5}" x="${link_5_x}" y="${link_5_y}" z="${link_5_z}"/>
+        <!-- <inertia
           ixx="0.0006353666666666666"
           ixy="0.0"
@@ -219,5 +268,5 @@
           iyy="0.0005020333333333333"
           iyz="0.0"
-          izz="0.00019333333333333333" />
+          izz="0.00019333333333333333" /> -->
       </inertial>
       <visual>
@@ -240,7 +289,7 @@
         </geometry>
       </collision>
-    </link> -->
+    </link>
     <!--Joint 5 ROLL JOINT-->
-    <!-- <joint name="${prefix}_joint_5" type="revolute">
+    <joint name="${prefix}_joint_5" type="revolute">
       <parent link="${prefix}_link_4"/>
       <child link="${prefix}_link_5"/>
@@ -250,11 +299,11 @@
         lower="-3.14159"
         upper="3.14159"
-        effort="2"
+        effort="1000"
         velocity="2" />
-      <dynamics damping="0.01" friction="0.5" />
-    </joint> -->
+      <!-- <dynamics damping="0.01" friction="0.5" /> -->
+    </joint>
     <!--PAD1 LINK-->
     <!-- Bounding box: 0.073966 0.02 0.01 -->
-    <!-- <link name="${prefix}_pad1_Link">
+    <link name="${prefix}_pad1_Link">
       <inertial>
         <origin
@@ -262,5 +311,5 @@
           rpy="0 0 0" />
         <mass
-          value="0.001" />
+          value="1.0" />
         <inertia
           ixx="4.166666666666667e-08"
@@ -294,7 +343,7 @@
         </geometry>
       </collision>
-    </link> -->
+    </link>
     <!--PAD1 JOINT-->
-    <!-- <joint  name="${prefix}_pad1_joint" type="revolute">
+    <joint  name="${prefix}_pad1_joint" type="revolute">
       <origin xyz="0 -0.0545 -0.0905" rpy="1.5708 -0.74758 -1.5708" />
       <parent link="${prefix}_link_5" />
@@ -304,11 +353,11 @@
         lower="0"
         upper="1.5709"
-        effort="1"
+        effort="1000"
         velocity="2" />
-      <dynamics damping="0.01" friction="0.01" />
-    </joint> -->
+      <!-- <dynamics damping="0.01" friction="0.01" /> -->
+    </joint>
     <!--PAD2 LINK-->
     <!-- Bounding box: 0.073966 0.02 0.01 -->
-    <!-- <link name="${prefix}_pad2_Link">
+    <link name="${prefix}_pad2_Link">
       <inertial>
         <origin
@@ -316,5 +365,5 @@
           rpy="0 0 0" />
         <mass
-          value="0.001" />
+          value="1.0" />
         <inertia
           ixx="4.166666666666667e-08"
@@ -348,7 +397,7 @@
         </geometry>
       </collision>
-    </link> -->
+    </link>
     <!--PAD2 JOINT-->
-    <!-- <joint name="${prefix}_pad2_joint" type="revolute">
+    <joint name="${prefix}_pad2_joint" type="revolute">
       <origin xyz="0 0.0545 -0.0905" rpy="-1.5708 -0.74758 1.5708" />
       <parent link="${prefix}_link_5" />
@@ -358,9 +407,9 @@
         lower="0"
         upper="1.5709"
-        effort="1"
+        effort="1000"
         velocity="2" />
-      <dynamics damping="0.01" friction="0.01" />
+      <!-- <dynamics damping="0.01" friction="0.01" /> -->
       <mimic joint="${prefix}_pad1_joint" multiplier="1.0" offset="0"/>
-    </joint> -->
+    </joint>
     <!-- Camera -->
     <!-- Bounding box: 0.089914 0.025 0.025055 -->
@@ -475,5 +524,5 @@
     </transmission>
     <!--Transmission Elbow-->
-    <!-- <transmission name="elbowTransmission">
+    <transmission name="elbowTransmission">
       <type>transmission_interface/SimpleTransmission</type>
       <joint name="${prefix}_joint_3" type="SimpleTransmission">
@@ -484,7 +533,7 @@
         <hardwareInterface>hardware_interface/PositionJointInterface</hardwareInterface>
       </actuator>
-    </transmission> -->
+    </transmission>
     <!--Transmission Pitch-->
-    <!-- <transmission name="pitchTransmission">
+    <transmission name="pitchTransmission">
       <type>transmission_interface/SimpleTransmission</type>
       <joint name="${prefix}_joint_4" type="SimpleTransmission">
@@ -495,7 +544,7 @@
         <hardwareInterface>hardware_interface/PositionJointInterface</hardwareInterface>
       </actuator>
-    </transmission> -->
+    </transmission>
     <!--Transmission Roll-->
-    <!-- <transmission name="pitchTransmission">
+    <transmission name="pitchTransmission">
       <type>transmission_interface/SimpleTransmission</type>
       <joint name="${prefix}_joint_5" type="SimpleTransmission">
@@ -506,7 +555,6 @@
         <hardwareInterface>hardware_interface/PositionJointInterface</hardwareInterface>
       </actuator>
-    </transmission> -->
+    </transmission>
     <!-- Transmission pad1-->
-<!--
     <transmission name="pad1Transmission">
       <type>transmission_interface/SimpleTransmission</type>
@@ -518,5 +566,5 @@
         <hardwareInterface>hardware_interface/PositionJointInterface</hardwareInterface>
       </actuator>
-    </transmission> -->
+    </transmission>
     <!-- Gazebo plugin for ROS Control -->
     <gazebo>
@@ -527,5 +575,5 @@
     <!-- Gazebo plugin MIMIC JOINT-->
     <!-- <robotNamespace>/scorbot</robotNamespace> -->
-    <!-- <gazebo>
+    <gazebo>
       <plugin name="mimic_pad1_joint" filename="libroboticsgroup_gazebo_mimic_joint_plugin.so">
         <joint>${prefix}_pad1_joint</joint>
@@ -537,7 +585,7 @@
         <maxEffort>10.0</maxEffort>
       </plugin>
-    </gazebo> -->
+    </gazebo>
     <!-- Gazebo plugin Grasp-->
-    <!-- <gazebo>
+    <gazebo>
       <plugin name="gazebo_grasp_fix" filename="libgazebo_grasp_fix.so">
         <arm>
@@ -555,5 +603,5 @@
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
Commit message: URDF updated: camera added

File: manipulation/scorbot_description/urdf/scorbot_v3.xacro (robot description, xacro)
@@ -354,5 +354,5 @@
     <!-- Camera -->
     <!-- Bounding box: 0.089914 0.025 0.025055 -->
-    <!-- <link name="camera_link">
+    <link name="camera_link">
       <inertial>
         <mass value="0.001"/>
@@ -376,11 +376,11 @@
         </geometry>
       </collision>
-    </link> -->
+    </link>
     <!-- Camera Joint -->
-    <!-- <joint name="camera_joint" type="fixed">
+    <joint name="camera_joint" type="fixed">
       <origin xyz="0.0 -0.07 0.0" rpy="${M_PI} 0 0" />
       <parent link="${prefix}_link_5"/>
       <child link="camera_link" />
-    </joint> -->
+    </joint>
     <!-- camera depth joints and links DONT INCLUDE STAY COMMENTED !!!!-->
     <!-- <joint name="camera_depth_joint" type="fixed">
@@ -391,19 +391,19 @@
     <link name="camera_depth_frame"/> -->
     <!-- Camera oriented -->
-    <!-- <joint name="camera_link_oriented_joint" type="fixed">
+    <joint name="camera_link_oriented_joint" type="fixed">
       <origin xyz="0 0 0" rpy="0 ${-M_PI/2} ${-M_PI/2}" />
       <parent link="camera_link" />
       <child link="camera_link_oriented" />
     </joint>
-    <link name="camera_link_oriented"/> -->
+    <link name="camera_link_oriented"/>
     <!-- Camera Depth Optical Frame -->
-    <!-- <joint name="camera_depth_optical_frame_joint" type="fixed">
+    <joint name="camera_depth_optical_frame_joint" type="fixed">
       <origin xyz="0 -0.0115 0" rpy="${-M_PI/2} 0 ${-M_PI/2}" />
       <parent link="camera_link_oriented" />
       <child link="camera_depth_optical_frame" />
     </joint>
-    <link name="camera_depth_optical_frame"/> -->
+    <link name="camera_depth_optical_frame"/>
     <!-- Camera plugin -->
-    <!-- <gazebo reference="camera_link_oriented">
+    <gazebo reference="camera_link_oriented">
       <sensor type="depth" name="camera_depth_sensor">
         <always_on>true</always_on>
@@ -440,5 +440,5 @@
         </plugin>
       </sensor>
-    </gazebo> -->
+    </gazebo>
     <!--Transmission Base -->
     <transmission name="baseTransmission">

Commit message: added pick place script using joint cmds

File: manipulation/scorbot_description/urdf/scorbot_v3.xacro (robot description, xacro)
@@ -14,4 +14,5 @@
   <xacro:property name="mass_pad1_Link" value="0.005" />
   <xacro:property name="mass_pad2_Link" value="0.005" />
+  <xacro:property name="mass_camera_link" value="0.001" />
   <!--Surrounding boxes values for each link-->
   <xacro:property name="base_link_x" value="0.24" />
@@ -39,4 +40,7 @@
   <xacro:property name="pad2_link_y" value="0.02" />
   <xacro:property name="pad2_link_z" value="0.01" />
+  <xacro:property name="camera_x" value="0.089914" />
+  <xacro:property name="camera_y" value="0.025" />
+  <xacro:property name="camera_z" value="0.025055" />
   <!--Inertia Calculator for a Box-->
   <xacro:macro name="box_inertia" params="mass x y z">
@@ -204,6 +208,6 @@
       <parent link="${prefix}_link_3"/>
       <child link="${prefix}_link_4"/>
-      <origin xyz="0.2225 0 0" rpy="0 0 0"/>
-      <axis xyz="0 0 1"/>
+      <origin xyz="0.2225 0 0" rpy="1.570796327 0 0"/>
+      <axis xyz="0 1 0"/>
       <limit lower="-2.268928" upper="2.268928" effort="1000" velocity="2"/>
       <!-- <dynamics
@@ -219,5 +223,5 @@
           rpy="0 0 0" />
         <mass
-          value="${mass_link_5}" />" />
+          value="${mass_link_5}"  />
         <xacro:box_inertia mass="${mass_link_5}" x="${link_5_x}" y="${link_5_y}" z="${link_5_z}"/>
       </inertial>
@@ -356,11 +360,7 @@
     <link name="camera_link">
       <inertial>
-        <mass value="0.001"/>
-        <origin xyz="0.0 0.0 -0.05" rpy="0 0 0"/>
-        <inertia
-          ixx="1.0439608541666666e-07" ixy="0.0" ixz="0.0"
-          iyy="7.260233684166666e-07" iyz="0.0"
-          izz="7.257939496666667e-07"
-          />
+        <origin xyz="0.0 0.0 0.0" rpy="0 0 0"/>
+        <mass value="${mass_camera_link}"/>
+        <xacro:box_inertia mass="${mass_camera_link}" x="${camera_x}" y="${camera_y}" z="${camera_z}"/>
       </inertial>
       <visual>
@@ -373,5 +373,6 @@
         <origin xyz="0 0 0" rpy="0 0 0"/>
         <geometry>
-          <box size="${d435_cam_width} ${d435_cam_depth} ${d435_cam_height}"/>
+          <mesh filename="package://rover_autonav/meshes/d435.dae"/>
+          <!-- <box size="${d435_cam_width} ${d435_cam_depth} ${d435_cam_height}"/> -->
         </geometry>
       </collision>
@@ -379,6 +380,6 @@
     <!-- Camera Joint -->
     <joint name="camera_joint" type="fixed">
-      <origin xyz="0.0 -0.07 0.0" rpy="${M_PI} 0 0" />
-      <parent link="${prefix}_link_5"/>
+      <origin xyz="0.0 0.0 0.07" rpy="${M_PI/2} 0 ${M_PI/2}" />
+      <parent link="${prefix}_link_4"/>
       <child link="camera_link" />
     </joint>
@@ -539,5 +540,5 @@
         <grip_count_threshold>1</grip_count_threshold>
         <max_grip_count>20</max_grip_count>
-        <release_tolerance>0.03</release_tolerance>
+        <release_tolerance>0.005</release_tolerance>
         <disable_collisions_on_attach>true</disable_collisions_on_attach>
         <contact_topic>__default_topic__</contact_topic>

Commit message: Manipulation pick_place_ee

File: manipulation/scorbot_description/urdf/scorbot_v3.xacro (robot description, xacro)
@@ -259,4 +259,12 @@
       <!-- <dynamics damping="0.01" friction="0.5" /> -->
     </joint>
+    <!--END EFFECTOR LINK-->
+    <link name="end_effector_link"/>
+    <!-- End effector Joint-->
+    <joint name="end_effector_joint" type="fixed">
+      <parent link="${prefix}_link_5" />
+      <child link = "end_effector_link" />
+      <origin xyz="0.0 0.0 -0.115" rpy="0.0 ${M_PI/2} 0.0" />
+    </joint>
     <!--PAD1 LINK-->
     <!-- Bounding box: 0.073966 0.02 0.01 -->

Commit message: Cleaning repo

File: manipulation/scorbot_description/urdf/scorbot_v3.xacro (robot description, xacro)
@@ -265,5 +265,5 @@
       <parent link="${prefix}_link_5" />
       <child link = "end_effector_link" />
-      <origin xyz="0.0 0.0 -0.115" rpy="0.0 ${M_PI/2} 0.0" />
+      <origin xyz="0.0 0.0 -0.14" rpy="0.0 ${M_PI/2} 0.0" />
     </joint>
     <!--PAD1 LINK-->
