Commit message: new update

File: manipulation/scorbot_description/urdf/scorbot_v3.xacro (robot description, xacro)
@@ -60,8 +60,10 @@
     <!--BASE LINK-->
     <!--Bounding box: 0.24 0.24 0.2274-->
+    <!--inertial : origin: xyz="0.0 0.0 0.11"-->
+    <!--inertial : origin: xyz="0.27 0.0 0.359"-->
     <link name="${prefix}_base_link">
       <inertial>
         <origin
-          xyz="0.0 0.0 0.11"
+          xyz="0.27 0.0 0.469"
           rpy="0 0 0" />
         <mass
@@ -265,5 +267,5 @@
       <parent link="${prefix}_link_5" />
       <child link = "end_effector_link" />
-      <origin xyz="0.0 0.0 -0.14" rpy="0.0 ${M_PI/2} 0.0" />
+      <origin xyz="0.0 0.0 -0.14" rpy="0.0 0.0 0.0" />
     </joint>
     <!--PAD1 LINK-->

File: rover_autonav/urdf/cali_urdf_complete_v3.xacro (robot description, xacro)
@@ -8,13 +8,15 @@
   <!-- <xacro:include filename="$(find rover_autonav)/urdf/rosbob_v2.xacro" /> -->
   <!-- MESH FOR MOBILE ROBOT-->
-  <xacro:include filename="$(find rover_autonav)/urdf/rosbob_v3.xacro" />
+  <xacro:include filename="$(find rover_autonav)/urdf/rosbob_v5.xacro" />
   <!-- ARM -->
   <xacro:include filename="$(find manipulation)/scorbot_description/urdf/scorbot_v3.xacro" />
   <!-- Here we create the Xacro macro to attach the Gripper to the arm_link-->
-  <xacro:scorbot prefix="scorbot" parent="arm_link">
+  <!-- <xacro:scorbot prefix="scorbot" parent="arm_link"> -->
+  <xacro:scorbot prefix="scorbot" parent="robot_footprint">
     <!-- NO MESH FOR MOBILE ROBOT-->
     <!-- <origin xyz="0.0 0 0.43" rpy="0 0 0" /> -->
     <!-- MESH FOR MOBILE ROBOT-->
-    <origin xyz="0.27 0 0.28" rpy="0 0 0" />
+    <!-- <origin xyz="0.27 0 0.28" rpy="0 0 0" /> -->
+    <origin xyz="0.27 0 0.359" rpy="0 0 0" />
   </xacro:scorbot>
 </robot>

File: rover_autonav/urdf/rosbob_v5.xacro (robot description, xacro)
@@ -14,4 +14,11 @@
 	<xacro:property name="pi" value="3.141592654"/>
 	<xacro:property name="half_pi" value="1.570796327"/>
+    <!--Inertia Calculator for a Box-->
+    <xacro:macro name="box_inertia" params="mass x y z">
+        <inertia  ixx="${mass*(y*y+z*z)/12.0}" ixy = "0" ixz = "0"
+              iyy="${mass*(x*x+z*z)/12.0}" iyz = "0"
+              izz="${mass*(x*x+y*y)/12.0}"
+        />
+    </xacro:macro>
 	<!-- Make Chassis of Bot -->
 	<link name="base_link">
@@ -20,9 +27,5 @@
 			<mass value="${robot_chassis_mass}"/>
       		<origin xyz="-0.05 0 0.3429" rpy=" 0 0 0"/>
-      		<inertia
-      			ixx="0.5806792822" ixy="0" ixz="0"
-      			iyy="1.705057074" iyz="0"
-      			izz="2.103962526"
-      		/>
+      		<xacro:box_inertia mass="${robot_chassis_mass}" x="${robot_chassis_length}" y="${robot_chassis_width}" z="${robot_chassis_height}"/>
 		</inertial>
 		<collision name="collision">
@@ -252,10 +255,10 @@
 	</joint>
 	<!-- JOIN ARM URDF !!!!!!!!!!!!!!!!!!-->
-	<joint name="arm_fixed_joint" type="fixed">
+	<!-- <joint name="arm_fixed_joint" type="fixed">
       <parent link="base_link" />
       <child link = "arm_link" />
       <origin xyz="0.0 0.0 0.0" rpy="0.0 0.0 0.0" />
-    </joint>
-    <link name="arm_link">
+    </joint> -->
+    <!-- <link name="arm_link">
       <collision>
         <geometry>
@@ -264,5 +267,5 @@
         <origin rpy="0 0 0" xyz="0 0 0"/>
       </collision>
-    </link>
+    </link> -->
 	<!-- Color of bot -->
 	<gazebo reference="left_wheel_front">
