Commit message: new update

File: rover_autonav/urdf/rosbob_v3.xacro (robot description, xacro)
@@ -1,5 +1,5 @@
 <?xml version='1.0'?>
-<robot name="rosbob" xmlns:xacro="http://www.ros.org/wiki/xacro">
-	<xacro:property name="robot_name" value="rosbob" />
+<robot name="cali" xmlns:xacro="http://www.ros.org/wiki/xacro">
+	<xacro:property name="robot_name" value="cali" />
 	<xacro:property name="robot_chassis_mass" value="34.5"/>
 	<xacro:property name="robot_chassis_length" value="0.7493"/>
@@ -7,6 +7,7 @@
     <xacro:property name="robot_chassis_height" value="0.1778"/>
 	<xacro:property name="robot_wheel_mass" value="1"/>
-	<xacro:property name="robot_wheel_length" value="0.112"/>
-	<xacro:property name="robot_wheel_radius" value="0.127"/>
+	<xacro:property name="robot_wheel_length" value="0.12"/>
+	<xacro:property name="robot_wheel_radius" value="0.16"/>
+	<!-- <xacro:property name="robot_wheel_radius" value="0.127"/> -->
 	<xacro:property name="camera_mass" value="0.1"/>
 	<xacro:property name="hokoyu_mass" value="1e-5"/>
@@ -15,5 +16,5 @@
 	<!-- Make Chassis of Bot -->
 	<link name="base_link">
-		<pose>0 0 0.1 0 0 0</pose>
+		<pose>0 0 0 0 0 0</pose>
 		<inertial>
 			<mass value="${robot_chassis_mass}"/>
@@ -232,5 +233,5 @@
 	<!-- Footprint joint-->
 	<joint name="robot_footprint_joint" type="fixed">
-		<origin xyz="0 0 0" rpy="0 0 0" />
+		<origin xyz="0 0 0.079" rpy="0 0 0" />
 		<parent link="robot_footprint"/>
 		<child link="base_link" />
@@ -245,5 +246,5 @@
 	<!-- Hokoyu Joint -->
 	<joint name="hokuyo_joint" type="fixed">
-	    <origin xyz="0.33 0 0.2" rpy="0 0 0" />
+	    <origin xyz="0.5 0 0.2" rpy="0 0 0" />
 	    <parent link="base_link"/>
 	    <child link="hokuyo" />
@@ -269,6 +270,6 @@
 		<kp>1000000.0</kp> <!-- kp and kd for rubber -->
 		<kd>100.0</kd>
-		<mu1>1.0</mu1>
-		<mu2>1.0</mu2>
+		<mu1>1000.0</mu1>
+		<mu2>1000.0</mu2>
 		<maxVel>1.0</maxVel>
 		<minDepth>0.00</minDepth>
@@ -278,6 +279,6 @@
 		<kp>1000000.0</kp> <!-- kp and kd for rubber -->
 		<kd>100.0</kd>
-		<mu1>1.0</mu1>
-		<mu2>1.0</mu2>
+		<mu1>1000.0</mu1>
+		<mu2>1000.0</mu2>
 		<maxVel>1.0</maxVel>
 		<minDepth>0.00</minDepth>
@@ -287,6 +288,6 @@
 		<kp>1000000.0</kp> <!-- kp and kd for rubber -->
 		<kd>100.0</kd>
-		<mu1>1.0</mu1>
-		<mu2>1.0</mu2>
+		<mu1>1000.0</mu1>
+		<mu2>1000.0</mu2>
 		<maxVel>1.0</maxVel>
 		<minDepth>0.00</minDepth>
@@ -296,6 +297,6 @@
 		<kp>1000000.0</kp> <!-- kp and kd for rubber -->
 		<kd>100.0</kd>
-		<mu1>1.0</mu1>
-		<mu2>1.0</mu2>
+		<mu1>1000.0</mu1>
+		<mu2>1000.0</mu2>
 		<maxVel>1.0</maxVel>
 		<minDepth>0.00</minDepth>

File: rover_autonav/urdf/rosbob_v4.xacro (robot description, xacro)
@@ -1,5 +1,5 @@
 <?xml version='1.0'?>
-<robot name="rosbob" xmlns:xacro="http://www.ros.org/wiki/xacro">
-	<xacro:property name="robot_name" value="rosbob" />
+<robot name="cali" xmlns:xacro="http://www.ros.org/wiki/xacro">
+	<xacro:property name="robot_name" value="cali" />
 	<xacro:property name="robot_chassis_mass" value="34.5"/>
 	<xacro:property name="robot_chassis_length" value="0.7493"/>
@@ -8,5 +8,5 @@
 	<xacro:property name="robot_wheel_mass" value="1"/>
 	<xacro:property name="robot_wheel_length" value="0.112"/>
-	<xacro:property name="robot_wheel_radius" value="0.127"/>
+	<xacro:property name="robot_wheel_radius" value="0.153"/>
 	<xacro:property name="camera_mass" value="0.1"/>
 	<xacro:property name="hokoyu_mass" value="1e-5"/>
@@ -18,5 +18,5 @@
 		<inertial>
 			<mass value="${robot_chassis_mass}"/>
-      		<origin xyz="0.0 0.3429" rpy=" 0 0 0"/>
+      		<origin xyz="-0.05 0 0.3429" rpy=" 0 0 0"/>
       		<inertia
       			ixx="0.5806792822" ixy="0" ixz="0"
@@ -43,5 +43,5 @@
 		<inertial>
 			<mass value="${robot_wheel_mass}"/>
-			<origin xyz="0 0 0" rpy="0 0 1.5707"/>
+			<origin xyz="0 0 0" rpy="1.5707 1.5707 -1.5707"/>
 			<inertia
 				ixx="0.005077583333333333" ixy="0.0" ixz="0.0"
@@ -58,5 +58,5 @@
 		</visual>
 		<collision>
-			<origin xyz="0 0 0" rpy="0 1.5707 1.5707"/>
+			<origin xyz="0 0 0" rpy="1.5707 0 0"/>
 			<geometry>
 				<cylinder radius="${robot_wheel_radius}" length="${robot_wheel_length}"/>
@@ -68,5 +68,5 @@
 		<inertial>
 			<mass value="${robot_wheel_mass}"/>
-			<origin xyz="0 0 0" rpy="0 1.5707 1.5707"/>
+			<origin xyz="0 0 0" rpy="1.5707 1.5707 -1.5707"/>
 			<inertia
 				ixx="0.005077583333333333" ixy="0.0" ixz="0.0"
@@ -83,5 +83,5 @@
 		</visual>
 		<collision>
-			<origin xyz="0 0 0" rpy="0 1.5707 1.5707"/>
+			<origin xyz="0 0 0" rpy="1.5707 0.0 0"/>
 			<geometry>
 				<cylinder radius="${robot_wheel_radius}" length="${robot_wheel_length}"/>
@@ -93,5 +93,5 @@
 		<inertial>
 			<mass value="${robot_wheel_mass}"/>
-			<origin xyz="0 0 0" rpy="0 1.5707 1.5707"/>
+			<origin xyz="0 0 0" rpy="1.5707 1.5707 -1.5707"/>
 			<inertia
 				ixx="0.005077583333333333" ixy="0.0" ixz="0.0"
@@ -101,5 +101,5 @@
 		</inertial>
 		<visual>
-			<origin xyz="0 0 0" rpy="1.5707 0.0 1.5707"/>
+			<origin xyz="0 0 0" rpy="1.5707 0.0 -1.5707"/>
 			<geometry>
 				<mesh filename="package://rover_autonav/meshes_v2/wheel.STL" />
@@ -108,5 +108,5 @@
 		</visual>
 		<collision>
-			<origin xyz="0 0 0" rpy="0 1.5707 1.5707"/>
+			<origin xyz="0 0 0" rpy="1.5707 0.0 0"/>
 			<geometry>
 				<cylinder radius="${robot_wheel_radius}" length="${robot_wheel_length}"/>
@@ -118,5 +118,5 @@
 		<inertial>
 			<mass value="${robot_wheel_mass}"/>
-			<origin xyz="0 0 0" rpy="0 1.5707 1.5707"/>
+			<origin xyz="0 0 0" rpy="1.5707 1.5707 -1.5707"/>
 			<inertia
 				ixx="0.005077583333333333" ixy="0.0" ixz="0.0"
@@ -126,5 +126,5 @@
 		</inertial>
 		<visual>
-			<origin xyz="0 0 0" rpy="1.5707 0.0 1.5707"/>
+			<origin xyz="0 0 0" rpy="1.5707 0.0 -1.5707"/>
 			<geometry>
 				<mesh filename="package://rover_autonav/meshes_v2/wheel.STL" />
@@ -133,5 +133,5 @@
 		</visual>
 		<collision>
-			<origin xyz="0 0 0" rpy="0 1.5707 1.5707"/>
+			<origin xyz="0 0 0" rpy="1.5707 0.0 0"/>
 			<geometry>
 				<cylinder radius="${robot_wheel_radius}" length="${robot_wheel_length}"/>
@@ -192,5 +192,5 @@
 	<!-- Right Wheel Joint Back-->
 	<joint type="continuous" name="right_wheel_hinge_back">
-	    <origin xyz="-0.38 -0.38 0.081" rpy="0 0 0" />
+	    <origin xyz="-0.38 -0.36785 0.081" rpy="0 0 0" />
 		<!-- <origin xyz="-0.37465 -0.313175 -0.2159" rpy="0 0 0" /> -->
 	    <parent link="base_link"/>
@@ -202,5 +202,5 @@
 	<!-- Right Wheel Joint Front-->
 	<joint type="continuous" name="right_wheel_hinge_front">
-	    <origin xyz="0.345 -0.38 0.081" rpy="0 0 0" />
+	    <origin xyz="0.345 -0.36785 0.081" rpy="0 0 0" />
 		<!-- <origin xyz="0.37465 -0.313175 -0.2159" rpy="0 0 0" /> -->
 	    <parent link="base_link"/>
@@ -212,5 +212,5 @@
 	<!-- Left Wheel Joint Back-->
 	<joint type="continuous" name="left_wheel_hinge_back">
-	    <origin xyz="-0.38 0.38 0.081" rpy="0 0 0" />
+	    <origin xyz="-0.38 0.36785 0.081" rpy="0 0 0" />
 		<!-- <origin xyz="-0.37465 0.313175 -0.2159" rpy="0 0 0" /> -->
 	    <parent link="base_link"/>
@@ -222,5 +222,5 @@
 	<!-- Left Wheel Joint Front-->
 	<joint type="continuous" name="left_wheel_hinge_front">
-	    <origin xyz="0.345 0.38 0.081" rpy="0 0 0" />
+	    <origin xyz="0.345 0.36785 0.081" rpy="0 0 0" />
 		<!-- <origin xyz="0.37465 0.313175 -0.2159" rpy="0 0 0" /> -->
 	    <parent link="base_link"/>
@@ -311,4 +311,4 @@
 	</gazebo>
 	<!-- Motor, Camera and Lidar Simulation -->
-	<xacro:include filename="$(find rover_autonav)/urdf/rosbob_v3.gazebo" />
+	<xacro:include filename="$(find rover_autonav)/urdf/rosbob_v4.gazebo" />
 </robot>
